File: CarBot_ModuleV2/CarBot_ModuleV2/CarBot_ModuleV2.kicad_sch (KiCad schematic)
At the start: 55 parts, among them J1 Line_Tracking, J10 Motor_A, J11 Motor_B, J12 RGB_LED, J2 Buck, J3 OLED, J4 Line_Tracking, J5 Batt_1, J6 Batt_2, J7 Barrel_Jack_Switch, J8 Ultrasonic, J9 TFT_Display, Q1 SS8050, Q2 AO3401A, SW1 B1, U1 TCRT5000_C, U2 TCRT5000_L, U3 TCRT5000_R, U6 AMS1117-3.3

Commit message: Finsh Layout V2
Parts:
- added H1, H2, H3, H4, H5, H6: MountingHole, MountingHole:MountingHole_3mm, symbol Mechanical:MountingHole
- BZ1: footprint (none) -> CarBotLibrary:Passive_Buzzer
- C1, C3, C5, C6: footprint (none) -> Capacitor_THT:C_Disc_D5.0mm_W2.5mm_P2.50mm
- C2: renamed from C7; footprint (none) -> Capacitor_THT:CP_Radial_D10.0mm_P3.80mm
- C4: renamed from C2; footprint (none) -> Capacitor_THT:C_Radial_D5.0mm_H11.0mm_P2.00mm; symbol Device:C_Small -> Device:C_Polarized
- C7: renamed from C4; footprint (none) -> Capacitor_THT:C_Radial_D5.0mm_H11.0mm_P2.00mm; symbol Device:C_Small -> Device:C_Polarized
- D2: footprint (none) -> LED_THT:LED_D3.0mm
- J1, J4: footprint (none) -> Connector_JST:JST_PH_B5B-PH-K_1x05_P2.00mm_Vertical
- J10, J11, J5, J6: footprint TerminalBlock_MetzConnect:TerminalBlock_MetzConnect_Type086_RT03402HBLC_1x02_P3.81mm_Horizontal -> CarBotLibrary:Pluggable Terminal Block 5.08-2P Right Angle
- J2: footprint (none) -> CarBotLibrary:Buck_farce
- J3, J8: footprint (none) -> Connector_PinHeader_2.54mm:PinHeader_1x04_P2.54mm_Vertical
- J7: footprint (none) -> Connector_BarrelJack:BarrelJack_Horizontal
- J9: footprint (none) -> Connector_PinHeader_2.54mm:PinHeader_1x08_P2.54mm_Vertical
- Q1, Q2: footprint Package_TO_SOT_SMD:SOT-23 -> Package_TO_SOT_SMD:SOT-23_Handsoldering
- U4: footprint (none) -> CarBotLibrary:ESP32-30pins
- U5: footprint (none) -> CarBotLibrary:MotDriver
- U6: renamed from U7; footprint Package_TO_SOT_SMD:SOT-23-6 -> Package_TO_SOT_SMD:SOT-23-6_Handsoldering
- U7: renamed from U8; footprint Package_TO_SOT_SMD:SOT-23-6 -> Package_TO_SOT_SMD:SOT-23-6_Handsoldering
- U9: footprint (none) -> CarBotLibrary:Switch SPDT 3PIN 3mm Pin spacing
- renumbered R12 to R11, R11 to R12, R21 to R18, R18 to R19, R19 to R20, R20 to R21, U6 to U8
Connections:
- net EN_M_A1: now also U4.9 (D26); no longer U4.6 (D32)
- net EN_M_A2: now also U4.8 (D25); no longer U4.7 (D33)
- net EN_M_B1: now also U4.7 (D33); no longer U4.8 (D25)
- net EN_M_B2: now also U4.6 (D32); no longer U4.9 (D26)

Commit message: Finsh car module V2
Parts:
- J1, J4: footprint Connector_JST:JST_PH_B5B-PH-K_1x05_P2.00mm_Vertical -> Connector_JST:JST_EH_B5B-EH-A_1x05_P2.50mm_Vertical
- J9: footprint Connector_PinHeader_2.54mm:PinHeader_1x08_P2.54mm_Vertical -> Connector_JST:JST_EH_B8B-EH-A_1x08_P2.50mm_Vertical
Changed lines of the file:
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@@
 			)
 		)
-		(property "Footprint" "Connector_PinHeader_2.54mm:PinHeader_1x08_P2.54mm_Vertical"
+		(property "Footprint" "Connector_JST:JST_EH_B8B-EH-A_1x08_P2.50mm_Vertical"
 			(at 271.145 112.395 0)
 			(effects
@@
 			)
 		)
-		(property "Footprint" "Connector_JST:JST_PH_B5B-PH-K_1x05_P2.00mm_Vertical"
+		(property "Footprint" "Connector_JST:JST_EH_B5B-EH-A_1x05_P2.50mm_Vertical"
 			(at 94.615 156.845 0)
 			(effects
@@
 			)
 		)
-		(property "Footprint" "Connector_JST:JST_PH_B5B-PH-K_1x05_P2.00mm_Vertical"
+		(property "Footprint" "Connector_JST:JST_EH_B5B-EH-A_1x05_P2.50mm_Vertical"
 			(at 267.97 133.985 0)
 			(effects
